File: EQM_1/secc_sch.kicad_sch (KiCad schematic)
At the start: 48 parts, among them J501 Screw_Terminal_01x05, SW401 SW_Push, SW402 SW_Push, U401 TL082, U402 CD4066BM

Commit message: PCB-1
Primer posicionamiento de los componentes en la pcb y ligeros cambios en el esquemático.
Posicionamiento MUY BASTO, simplemente para ver que los componentes caben en las dimensiones de la pcb elegida.
Parts:
- C401, C402, C404, C405, C406: value C -> 100nF; footprint (none) -> Capacitor_SMD:C_0805_2012Metric_Pad1.18x1.45mm_HandSolder
- D401, D402, D501: footprint (none) -> Diode_SMD:D_0805_2012Metric_Pad1.15x1.40mm_HandSolder
- J406, J407: footprint (none) -> Connector_PinHeader_2.54mm:PinHeader_1x03_P2.54mm_Vertical
- J501: footprint (none) -> TerminalBlock_Phoenix:TerminalBlock_Phoenix_MKDS-1,5-5-5.08_1x05_P5.08mm_Horizontal
- R401, R406, R407, R408: value R -> 10K; footprint (none) -> Resistor_SMD:R_0805_2012Metric_Pad1.20x1.40mm_HandSolder
- R401: value R -> 10K; footprint (none) -> Resistor_THT:R_Axial_DIN0207_L6.3mm_D2.5mm_P7.62mm_Horizontal
- R401, R406: value R -> 670R; footprint (none) -> Resistor_SMD:R_0805_2012Metric_Pad1.20x1.40mm_HandSolder
- SW401, SW402: footprint (none) -> Button_Switch_SMD:SW_Tactile_SPST_NO_Straight_CK_PTS636Sx25SMTRLFS; digikeyPN (none) -> CKN12314-2-ND; digikeyURL (none) -> https://www.digikey.com/en/products/detail/c-k/PTS636-SM50-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
- TP301: footprint (none) -> TestPoint:TestPoint_Pad_2.0x2.0mm
- U401: footprint (none) -> Package_TO_SOT_SMD:SOT-23-8
Connections:
- net CS_{1}: now also J406.1; no longer J406.2
- net CS_{2}: now also J407.1; no longer J407.2
- net CS_{3}: now also J406.1; no longer J406.2
- net CS_{4}: now also J407.1; no longer J407.2
- net V_{Control-1}: now also J406.2; no longer J406.1
- net V_{Control-2}: now also J407.2; no longer J407.1
- net V_{Control-3}: now also J406.2; no longer J406.1
- net V_{Control-4}: now also J407.2; no longer J407.1
- net #VSS renamed VSS
Other:
- moved on the sheet: C405, C406, R407, R408, SW401, SW402
